File: Documentation/KiCAD/HgMJK_N-bane_Turntable/HgMJK_N-bane_Turntable.kicad_sch (KiCad schematic)
At the start: 10 parts, among them J1 Screw_Terminal_01x02, M1 Stepper_Motor_unipolar_5pin, SW2 SW_DPST_x2, U1 ULN2003

Commit message: file update - KiCAD
updated - KiCAD sch. Deleted old KiCAD backup files
Connections:
- net +12V: now also M1.1
- net at U1.13 (O4): now also M1.5
- net at U1.14 (O3): now also M1.4
- net at U1.15 (O2): now also M1.3 (-)
- net at U1.16 (O1): now also M1.2
Other:
- moved on the sheet: M1
Changed lines of the file:
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@@
 	(symbol
 		(lib_id "Motor:Stepper_Motor_unipolar_5pin")
-		(at 185.42 66.04 0)
+		(at 201.93 123.19 0)
 		(unit 1)
 		(exclude_from_sim no)
@@
 		(dnp no)
 		(property "Reference" "M1"
-			(at 190.5 63.792 0)
+			(at 207.01 120.942 0)
 			(effects
 				(font
@@
 		)
 		(property "Value" "Stepper_Motor_unipolar_5pin"
-			(at 178.308 71.12 0)
+			(at 194.818 128.27 0)
 			(effects
 				(font
@@
 		)
 		(property "Footprint" ""
-			(at 185.674 66.294 0)
+			(at 202.184 123.444 0)
 			(effects
 				(font
@@
 		)
 		(property "Datasheet" "http://www.infineon.com/dgdl/Application-Note-TLE8110EE_driving_UniPolarStepperMotor_V1.1.pdf?fileId=db3a30431be39b97011be5d0aa0a00b0"
-			(at 185.674 66.294 0)
+			(at 202.184 123.444 0)
 			(effects
 				(font
@@
 		)
 		(property "Description" "5-wire unipolar stepper motor"
-			(at 185.42 66.04 0)
+			(at 201.93 123.19 0)
 			(effects
 				(font
